File: PCB/peedee/peedee.kicad_pcb (KiCad board)
At the start: 2 copper layers, 16 x 42.5 mm, 17 parts, among them J2 Conn_02x05_Odd_Even, SW1 TIMR-05-T-V-T/R, U1 10k, U2 CH224K, U3 10k, U4 10k, U5 10k

Commit message: Update peedee.kicad_pcb
Routing:
- net /VBUS: track 15.9 -> 13.6 mm
Changed lines of the file:
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@@
 	)
 	(segment
-		(start 134.2 47.8)
-		(end 133.8 47.2)
-		(width 0.5)
-		(layer "F.Cu")
-		(net "/VBUS")
-	)
-	(segment
-		(start 134.205882 48.205882)
-		(end 135.194118 48.205882)
+		(start 134.4 48.1)
+		(end 134.205882 48.205882)
 		(width 0.5)
 		(layer "F.Cu")
@@
 		(start 142.2 48.2)
 		(end 143.457107 48.2)
+		(width 0.5)
+		(layer "F.Cu")
+		(net "/VBUS")
+	)
+	(segment
+		(start 134.8 48.1)
+		(end 134.4 48.1)
 		(width 0.5)
 		(layer "F.Cu")
@@
 	)
 	(segment
-		(start 135.194118 48.205882)
-		(end 135.3 48.1)
-		(width 0.5)
-		(layer "F.Cu")
-		(net "/VBUS")
-	)
-	(segment
 		(start 135.3 48.1)
 		(end 136.3275 48.1)
@@
 		(start 141.6 47.7)
 		(end 141.6 47.07)
-		(width 0.5)
-		(layer "F.Cu")
-		(net "/VBUS")
-	)
-	(segment
-		(start 134.4 48.1)
-		(end 134.205882 48.205882)
-		(width 0.5)
-		(layer "F.Cu")
-		(net "/VBUS")
-	)
-	(segment
-		(start 134.2 47.8)
-		(end 134.35 47.95)
-		(width 0.5)
-		(layer "F.Cu")
-		(net "/VBUS")
-	)
-	(segment
-		(start 134.8 48.1)
-		(end 134.4 48.1)
 		(width 0.5)
 		(layer "F.Cu")
@@
 	)
 	(segment
-		(start 134.205882 48.205882)
-		(end 133.3 48.7)
+		(start 135.194118 48.205882)
+		(end 135.3 48.1)
 		(width 0.5)
 		(layer "F.Cu")
@@
 	)
 	(segment
-		(start 134.4 48.1)
-		(end 134.2 47.8)
+		(start 134.205882 48.205882)
+		(end 135.194118 48.205882)
 		(width 0.5)
 		(layer "F.Cu")
