File: PCB/peedee/peedee.kicad_sch (KiCad schematic)
At the start: 17 parts, among them J2 Conn_02x05_Odd_Even, SW1 TIMR-05-T-V-T/R, U1 10k, U2 CH224K, U3 10k, U4 10k, U5 10k

Commit message: all the docs
Parts:
- C1: LCSC Part C29936 -> C1592; MPN CL10B105KA8NNNC -> CL10A105KO8NNNC
Changed lines of the file:
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@@
 			)
 		)
-		(property "Datasheet" "https://lcsc.com/product-detail/Multilayer-Ceramic-Capacitors-MLCC-SMD-SMT_SAMSUNG_CL10B105KA8NNNC_1uF-105-10-25V-X7R_C29936.html"
+		(property "Datasheet" ""
 			(at 142.24 39.37 0)
 			(hide yes)
@@
 			)
 		)
-		(property "Description" "1uF (105) ±10% 25V X7R"
+		(property "Description" "16V 1uF X5R ±10% 0603 Multilayer Ceramic Capacitors MLCC - SMD/SMT ROHS"
 			(at 132.08 39.37 0)
 			(hide yes)
@@
 			)
 		)
-		(property "MPN" "CL10B105KA8NNNC"
+		(property "MPN" "CL10A105KO8NNNC"
 			(at 147.32 39.37 0)
 			(hide yes)
@@
 			)
 		)
-		(property "LCSC Part" "C29936"
+		(property "LCSC Part" "C1592"
 			(at 149.86 39.37 0)
 			(hide yes)
